File: pcb/Flick.kicad_pcb (KiCad board)
At the start: 2 copper layers, 23.5 x 16.5 mm, 37 parts, among them Q1 SS8050, SW1 HX 3X4X2-2P, SW2 HX 3X4X2-2P, SW3 HX 3X4X2-2P, U1 PFS154-S08

Commit message: change component
Parts:
- D1: value IR204A -> IR333-A_C264290; footprint LED_THT:LED_D5.0mm_IRBlack -> lcsc_footprints:C264290_LED-TH_BD6_2-P2_54-FD
- moved D1 1.25 mm to (130.0, 68.8), turned to 180 degrees
- renumbered + to BAT+1, - to BAT-1
Connections:
- D1 pad 1: Net-(D1-K) -> Net-(D1-A)
- D1 pad 2: Net-(D1-A) -> Net-(D1-C)
- Q1 pad 3: Net-(D1-K) -> Net-(D1-C)
Routing:
- net Net-(D1-K): track 3.36 -> 0.00 mm
- net Net-(D1-C): track 0.00 -> 2.87 mm
- net Net-(D1-A): track 2.78 -> 2.27 mm
Changed lines of the file:
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@@
 			(layers "F.Cu" "F.Mask" "F.Paste")
 			(roundrect_rratio 0.25)
-			(net "Net-(D1-K)")
+			(net "Net-(D1-C)")
 			(pinfunction "C_3")
 			(pintype "passive")
@@
 		)
 	)
-	(footprint "LED_THT:LED_D5.0mm_IRBlack"
+	(footprint "lcsc_footprints:C264290_LED-TH_BD6_2-P2_54-FD"
 		(layer "F.Cu")
-		(at 128.725 68.75)
-		(descr "LED, diameter 5.0mm, 2 pins, infrared, black, http://cdn-reichelt.de/documents/datenblatt/A500/LL-504BC2E-009.pdf, generated by kicad-footprint-generator")
-		(tags "LED IR")
+		(at 129.98 68.75 180)
 		(property "Reference" "D1"
-			(at 1.275 -1.5 0)
+			(at 0 -4 0)
 			(layer "F.SilkS")
 			(effects
 				(font
-					(size 0.7 0.7)
-					(thickness 0.12)
+					(size 1 1)
+					(thickness 0.15)
 				)
 			)
 		)
-		(property "Value" "IR204A"
-			(at 1.27 3.96 0)
+		(property "Value" "IR333-A_C264290"
+			(at 0 4 0)
 			(layer "F.Fab")
 			(effects
 				(font
-					(size 0.7 0.7)
-					(thickness 0.12)
+					(size 1 1)
+					(thickness 0.15)
 				)
 			)
 		)
-		(property "Datasheet" "http://www.everlight.com/file/ProductFile/IR204-A.pdf"
+		(property "Datasheet" "https://www.lcsc.com/datasheet/lcsc_datasheet_1808280419_Everlight-Elec-IR333-A_C264290.pdf"
 			(at 0 0 0)
 			(layer "F.Fab")
@@
 			)
 		)
-		(property "Description" "Infrared LED , 3mm LED package"
+		(property "Description" "IR333-A_C264290"
 			(at 0 0 0)
 			(layer "F.Fab")
@@
 			)
 		)
-		(property "KiLib_Generator" "LED/THT"
+		(property "LCSC Part" "C264290"
 			(at 0 0 0)
-			(layer "F.SilkS")
+			(layer "F.Fab")
+			(hide yes)
+			(effects
+				(font
+					(size 1.27 1.27)
+				)
+			)
+		)
+		(property "LCSC" "C264290"
+			(at 0 0 180)
+			(unlocked yes)
+			(layer "F.Fab")
+			(hide yes)
+			(effects
+				(font
+					(size 1 1)
+					(thickness 0.15)
+				)
+			)
+		)
+		(property "Manufacturer" "EVERLIGHT(亿光)"
+			(at 0 0 180)
+			(unlocked yes)
+			(layer "F.Fab")
 			(hide yes)
 			(effects
@@
 			)
 		)
-		(property ki_fp_filters "LED*3.0mm*IRBlack*")
 		(sheetname "/")
 		(sheetfile "Flick.kicad_sch")
@@
 		(duplicate_pad_numbers_are_jumpers no)
 		(fp_line
-			(start -1.29 -1.545)
-			(end -1.29 1.545)
+			(start 2.92 -1.4)
+			(end 2.92 1.4)
 			(stroke
-				(width 0.12)
+				(width 0.25)
 				(type solid)
 			)
 			(layer "F.SilkS")
 		)
-		(fp_arc
-			(start -1.29 -1.54483)
-			(mid 2.071779 -2.880495)
-			(end 4.26 0)
+		(fp_line
+			(start -1.01 -1.04)
+			(end -1.01 -1.8)
 			(stroke
-				(width 0.12)
+				(width 0.25)
 				(type solid)
 			)
 			(layer "F.SilkS")
 		)
-		(fp_arc
-			(start 4.26 0)
-			(mid 2.071779 2.880495)
-			(end -1.29 1.54483)
+		(fp_line
+			(start -1.27 0.13)
+			(end -1.27 -0.63)
 			(stroke
-				(width 0.12)
+				(width 0.25)
 				(type solid)
 			)
 			(layer "F.SilkS")
 		)
-		(fp_circle
-			(center 1.27 0)
-			(end 3.77 0)
+		(fp_line
+			(start -1.39 -1.42)
+			(end -0.62 -1.42)
 			(stroke
-				(width 0.12)
+				(width 0.25)
 				(type solid)
 			)
-			(fill no)
 			(layer "F.SilkS")
 		)
-		(fp_rect
-			(start -1.94 -3.21)
-			(end 4.49 3.21)
+		(fp_line
+			(start -1.65 -0.25)
+			(end -0.89 -0.25)
 			(stroke
-				(width 0.05)
+				(width 0.25)
 				(type solid)
 			)
-			(fill no)
-			(layer "F.CrtYd")
+			(layer "F.SilkS")
 		)
-		(fp_line
-			(start -1.23 -1.469694)
-			(end -1.23 1.469694)
+		(fp_arc
+			(start 2.92 1.4)
+			(mid -3.124274 -0.000958)
+			(end 2.920842 -1.398279)
 			(stroke
-				(width 0.1)
+				(width 0.25)
 				(type solid)
 			)
-			(layer "F.Fab")
+			(layer "F.SilkS")
 		)
-		(fp_arc
-			(start -1.23 -1.469694)
-			(mid 4.17 0)
-			(end -1.23 1.469694)
+		(fp_circle
+			(center 0 0)
+			(end 2.5 0)
 			(stroke
-				(width 0.1)
+				(width 0.25)
 				(type solid)
 			)
-			(layer "F.Fab")
+			(fill no)
+			(layer "F.SilkS")
 		)
 		(fp_circle
-			(center 1.27 0)
-			(end 3.77 0)
+			(center -3.1 3.11)
+			(end -3.07 3.11)
 			(stroke
-				(width 0.1)
+				(width 0.06)
 				(type solid)
 			)
 			(fill no)
-			(layer "F.Fab")
+			(layer "F.SilkS")
+		)
+		(fp_line
+			(start 3.1 0)
+			(end -3.1 0)
+			(stroke
+				(width 0.05)
+				(type solid)
+			)
+			(layer "F.CrtYd")
+		)
+		(fp_line
+			(start -3.1 0)
+			(end 3.1 0)
+			(stroke
+				(width 0.05)
+				(type solid)
+			)
+			(layer "F.CrtYd")
 		)
 		(fp_text user "${REFERENCE}"
-			(at 1.27 0 0)
+			(at 0 0 0)
 			(layer "F.Fab")
 			(effects
 				(font
-					(size 0.7 0.7)
-					(thickness 0.12)
+					(size 1 1)
+					(thickness 0.15)
 				)
 			)
 		)
-		(point
-			(at 129.995 68.75)
-			(size 2)
-			(layer "F.Fab")
-		)
-		(pad "1" thru_hole rect
-			(at 0 0)
-			(size 1.8 1.8)
-			(drill 0.9)
+		(pad "1" thru_hole circle
+			(at -1.27 0 180)
+			(size 1.524 1.524)
+			(drill 0.9144)
 			(layers "*.Cu" "*.Mask")
 			(remove_unused_layers no)
-			(net "Net-(D1-K)")
-			(pinfunction "K_1")
-			(pintype "passive")
+			(net "Net-(D1-A)")
+			(pinfunction "A_1")
+			(pintype "input")
 		)
-		(pad "2" thru_hole circle
-			(at 2.54 0)
-			(size 1.8 1.8)
-			(drill 0.9)
+		(pad "2" thru_hole rect
+			(at 1.27 0 180)
+			(size 1.524 1.524)
+			(drill 0.9144)
 			(layers "*.Cu" "*.Mask")
 			(remove_unused_layers no)
-			(net "Net-(D1-A)")
-			(pinfunction "A_2")
-			(pintype "passive")
+			(net "Net-(D1-C)")
+			(pinfunction "C_2")
+			(pintype "input")
+			(thermal_bridge_angle 45)
 		)
 		(embedded_fonts no)
-		(model "${KICAD10_3DMODEL_DIR}/LED_THT.3dshapes/LED_D5.0mm_IRBlack.step"
+		(model "${KIPRJMOD}/libs/lcsc/3dmodels/C264290.wrl"
 			(offset
 				(xyz 0 0 0)
@@
 		(sheetname "/")
 		(sheetfile "Flick.kicad_sch")
+		(units
+			(unit
+				(name "A")
+				(pins "2" "1")
+			)
+		)
 		(attr through_hole)
 		(duplicate_pad_numbers_are_jumpers no)
@@
 		(descr "Keystone SMT Micro Mini Test Point 5015, http://www.keyelco.com/product-pdf.cfm?p=1353")
 		(tags "Test Point")
-		(property "Reference" "-"
+		(property "Reference" "BAT-1"
 			(at -0.044583 -2.461811 155)
 			(layer "B.Paste")
@@
 		(descr "Keystone SMT Micro Mini Test Point 5015, http://www.keyelco.com/product-pdf.cfm?p=1353")
 		(tags "Test Point")
-		(property "Reference" "+"
+		(property "Reference" "BAT+1"
 			(at 0.044583 -2.461811 205)
 			(layer "B.Paste")
@@
 	)
 	(segment
-		(start 129.3 71.375)
-		(end 129.3 70.3)
-		(width 0.6)
-		(layer "F.Cu")
-		(net "Net-(D1-K)")
-	)
-	(segment
-		(start 129.3 70.3)
-		(end 128.725 69.725)
-		(width 0.6)
-		(layer "F.Cu")
-		(net "Net-(D1-K)")
-	)
-	(segment
-		(start 128.725 69.725)
-		(end 128.725 68.25)
-		(width 0.6)
-		(layer "F.Cu")
-		(net "Net-(D1-K)")
-	)
-	(segment
 		(start 138.1375 70.75)
 		(end 138.1375 71.6125)
@@
 	)
 	(segment
-		(start 130.5875 68.9275)
-		(end 131.265 68.25)
+		(start 130.5875 69.4125)
+		(end 131.25 68.75)
 		(width 0.6)
 		(layer "F.Cu")
@@
 	(segment
 		(start 130.5875 70.75)
-		(end 130.5875 68.9275)
+		(end 130.5875 69.4125)
 		(width 0.6)
 		(layer "F.Cu")
@@
 		(net "Net-(R1-Pad2)")
 	)
+	(segment
+		(start 128.725 69.725)
+		(end 128.725 68.765)
+		(width 0.6)
+		(layer "F.Cu")
+		(net "Net-(D1-C)")
+	)
+	(segment
+		(start 128.725 68.765)
+		(end 128.71 68.75)
+		(width 0.6)
+		(layer "F.Cu")
+		(net "Net-(D1-C)")
+	)
+	(segment
+		(start 129.3 70.3)
+		(end 128.725 69.725)
+		(width 0.6)
+		(layer "F.Cu")
+		(net "Net-(D1-C)")
+	)
+	(segment
+		(start 129.3 71.375)
+		(end 129.3 70.3)
+		(width 0.6)
+		(layer "F.Cu")
+		(net "Net-(D1-C)")
+	)
 	(zone

Commit message: fix + parts list
Parts:
- renumbered BAT-1 to TP7, BAT+1 to TP8
Other:
- board text added: "+"
- board text added: "-"
Changed lines of the file:
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@@
 				(font
 					(size 1.27 1.27)
+					(thickness 0.15)
 				)
 			)
@@
 		(descr "Keystone SMT Micro Mini Test Point 5015, http://www.keyelco.com/product-pdf.cfm?p=1353")
 		(tags "Test Point")
-		(property "Reference" "BAT-1"
+		(property "Reference" "TP7"
 			(at -0.044583 -2.461811 155)
 			(layer "B.Paste")
+			(hide yes)
 			(effects
 				(font
@@
 		(descr "Keystone SMT Micro Mini Test Point 5015, http://www.keyelco.com/product-pdf.cfm?p=1353")
 		(tags "Test Point")
-		(property "Reference" "BAT+1"
+		(property "Reference" "TP8"
 			(at 0.044583 -2.461811 205)
 			(layer "B.Paste")
+			(hide yes)
 			(effects
 				(font
@@
 		(layer "Edge.Cuts")
 	)
+	(gr_text "+"
+		(at 130.5 77.5 25)
+		(layer "B.Paste")
+		(effects
+			(font
+				(size 1.5 1.5)
+				(thickness 0.375)
+				(bold yes)
+			)
+			(justify mirror)
+		)
+	)
+	(gr_text "-"
+		(at 148 77.5 335)
+		(layer "B.Paste")
+		(effects
+			(font
+				(size 1.5 1.5)
+				(thickness 0.375)
+				(bold yes)
+			)
+			(justify mirror)
+		)
+	)
 	(segment
 		(start 128.35 73.25)
@@
 	)
 	(segment
+		(start 128.725 69.725)
+		(end 128.725 68.765)
+		(width 0.6)
+		(layer "F.Cu")
+		(net "Net-(D1-C)")
+	)
+	(segment
+		(start 128.725 68.765)
+		(end 128.71 68.75)
+		(width 0.6)
+		(layer "F.Cu")
+		(net "Net-(D1-C)")
+	)
+	(segment
+		(start 129.3 70.3)
+		(end 128.725 69.725)
+		(width 0.6)
+		(layer "F.Cu")
+		(net "Net-(D1-C)")
+	)
+	(segment
+		(start 129.3 71.375)
+		(end 129.3 70.3)
+		(width 0.6)
+		(layer "F.Cu")
+		(net "Net-(D1-C)")
+	)
+	(segment
 		(start 138.1375 70.75)
 		(end 138.1375 71.6125)
@@
 		(net "Net-(R1-Pad2)")
 	)
-	(segment
-		(start 128.725 69.725)
-		(end 128.725 68.765)
-		(width 0.6)
-		(layer "F.Cu")
-		(net "Net-(D1-C)")
-	)
-	(segment
-		(start 128.725 68.765)
-		(end 128.71 68.75)
-		(width 0.6)
-		(layer "F.Cu")
-		(net "Net-(D1-C)")
-	)
-	(segment
-		(start 129.3 70.3)
-		(end 128.725 69.725)
-		(width 0.6)
-		(layer "F.Cu")
-		(net "Net-(D1-C)")
-	)
-	(segment
-		(start 129.3 71.375)
-		(end 129.3 70.3)
-		(width 0.6)
-		(layer "F.Cu")
-		(net "Net-(D1-C)")
-	)
 	(zone
