File: pcb/Flick.kicad_sch (KiCad schematic)
At the start: 37 parts, among them Q1 SS8050, SW1 HX 3X4X2-2P, SW2 HX 3X4X2-2P, SW3 HX 3X4X2-2P, U1 PFS154-S08

Commit message: change component
Parts:
- D1: value IR204A -> IR333-A_C264290; footprint LED_THT:LED_D5.0mm_IRBlack -> lcsc_footprints:C264290_LED-TH_BD6_2-P2_54-FD; symbol LED:IR204A -> lcsc_imported:IR333-A_C264290; LCSC (none) -> C264290; Manufacturer (none) -> EVERLIGHT(亿光)
Connections:
- net at Q1.3 (C): now also D1.2 (C); no longer D1.1 (K)
- net at R5.1: now also D1.1 (A); no longer D1.2 (A)
Other:
- moved on the sheet: R5
Changed lines of the file:
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@@
 	(wire
 		(pts
+			(xy 60.96 132.08) (xy 57.15 132.08)
+		)
+		(stroke
+			(width 0)
+			(type default)
+		)
+	)
+	(wire
+		(pts
 			(xy 133.35 81.28) (xy 138.43 81.28)
 		)
@@
 	(symbol
 		(lib_id "power:+3.3V")
-		(at 62.23 132.08 270)
+		(at 68.58 132.08 270)
 		(unit 1)
 		(body_style 1)
@@
 		(fields_autoplaced yes)
 		(property "Reference" "#PWR021"
-			(at 58.42 132.08 0)
+			(at 64.77 132.08 0)
 			(hide yes)
 			(show_name no)
@@
 		)
 		(property "Value" "+3.3V"
-			(at 66.04 132.0799 90)
+			(at 72.39 132.0799 90)
 			(show_name no)
 			(do_not_autoplace no)
@@
 		)
 		(property "Footprint" ""
-			(at 62.23 132.08 0)
+			(at 68.58 132.08 0)
 			(hide yes)
 			(show_name no)
@@
 		)
 		(property "Datasheet" ""
-			(at 62.23 132.08 0)
+			(at 68.58 132.08 0)
 			(hide yes)
 			(show_name no)
@@
 		)
 		(property "Description" "Power symbol creates a global label with name \"+3.3V\""
-			(at 62.23 132.08 0)
+			(at 68.58 132.08 0)
 			(hide yes)
 			(show_name no)
@@
 	(symbol
 		(lib_id "Device:R")
-		(at 58.42 132.08 90)
+		(at 64.77 132.08 90)
 		(unit 1)
 		(body_style 1)
@@
 		(fields_autoplaced yes)
 		(property "Reference" "R5"
-			(at 58.42 125.73 90)
+			(at 64.77 125.73 90)
 			(show_name no)
 			(do_not_autoplace no)
@@
 		)
 		(property "Value" "22 Om"
-			(at 58.42 128.27 90)
+			(at 64.77 128.27 90)
 			(show_name no)
 			(do_not_autoplace no)
@@
 		)
 		(property "Footprint" "Resistor_SMD:R_0603_1608Metric_Pad0.98x0.95mm_HandSolder"
-			(at 58.42 133.858 90)
+			(at 64.77 133.858 90)
 			(hide yes)
 			(show_name no)
@@
 		)
 		(property "Datasheet" ""
-			(at 58.42 132.08 0)
+			(at 64.77 132.08 0)
 			(hide yes)
 			(show_name no)
@@
 		)
 		(property "Description" "Resistor"
-			(at 58.42 132.08 0)
+			(at 64.77 132.08 0)
 			(hide yes)
 			(show_name no)
@@
 	)
 	(symbol
-		(lib_id "LED:IR204A")
-		(at 52.07 132.08 0)
+		(lib_id "lcsc_imported:IR333-A_C264290")
+		(at 52.07 132.08 180)
 		(unit 1)
 		(body_style 1)
@@
 		(fields_autoplaced yes)
 		(property "Reference" "D1"
-			(at 50.927 124.46 0)
+			(at 51.943 125.73 0)
+			(show_name no)
+			(do_not_autoplace no)
+			(effects
+				(font
+					(size 1.27 1.27)
+				)
+			)
+		)
+		(property "Value" "IR333-A_C264290"
+			(at 51.943 128.27 0)
+			(show_name no)
+			(do_not_autoplace no)
+			(effects
+				(font
+					(size 1.27 1.27)
+				)
+			)
+		)
+		(property "Footprint" "lcsc_footprints:C264290_LED-TH_BD6_2-P2_54-FD"
+			(at 52.07 121.92 0)
+			(hide yes)
 			(show_name no)
 			(do_not_autoplace no)
@@
 			)
 		)
-		(property "Value" "IR204A"
-			(at 50.927 127 0)
+		(property "Datasheet" "https://www.lcsc.com/datasheet/lcsc_datasheet_1808280419_Everlight-Elec-IR333-A_C264290.pdf"
+			(at 54.356 132.207 0)
+			(hide yes)
 			(show_name no)
 			(do_not_autoplace no)
@@
 			)
 		)
-		(property "Footprint" "LED_THT:LED_D5.0mm_IRBlack"
-			(at 52.07 127.635 0)
+		(property "Description" "IR333-A_C264290"
+			(at 52.07 132.08 0)
 			(hide yes)
 			(show_name no)
@@
 			)
 		)
-		(property "Datasheet" "http://www.everlight.com/file/ProductFile/IR204-A.pdf"
-			(at 50.8 132.08 0)
+		(property "LCSC" "C264290"
+			(at 52.07 132.08 0)
 			(hide yes)
 			(show_name no)
@@
 			)
 		)
-		(property "Description" "Infrared LED , 3mm LED package"
+		(property "Manufacturer" "EVERLIGHT(亿光)"
 			(at 52.07 132.08 0)
 			(hide yes)

Commit message: fix + parts list
Parts:
- renumbered BAT-1 to TP7, BAT+1 to TP8
Changed lines of the file:
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@@
 		(dnp no)
 		(fields_autoplaced yes)
-		(property "Reference" "BAT-1"
+		(property "Reference" "TP7"
 			(at 194.818 58.42 90)
 			(show_name no)
@@
 			(project "Flick"
 				(path "/a688768b-2e23-46b9-a667-3b762413612a"
-					(reference "BAT-1")
+					(reference "TP7")
 					(unit 1)
 				)
@@
 		(dnp no)
 		(fields_autoplaced yes)
-		(property "Reference" "BAT+1"
+		(property "Reference" "TP8"
 			(at 194.818 50.8 90)
 			(show_name no)
@@
 			(project "Flick"
 				(path "/a688768b-2e23-46b9-a667-3b762413612a"
-					(reference "BAT+1")
-					(unit 1)
-				)
+					(reference "TP8")
+					(unit 1)
+				)
